File: zx_splicer.sch (KiCad schematic (older format))
At the start: 8 parts, among them J1 Conn_02x04_Row_Letter_First, J2 Conn_02x23_Row_Letter_First, J3 Conn_02x04_Row_Letter_First, J4 Conn_02x23_Row_Letter_First, J5 Conn_02x04_Row_Letter_First, J6 Conn_02x23_Row_Letter_First, J7 Conn_02x04_Row_Letter_First, J8 Conn_02x23_Row_Letter_First

Commit message: Rename to ZX Splicer
Parts:
- J1: footprint zx_bus_breakout:short_board_socket -> zx_splicer:short_board_socket
- J2: footprint zx_bus_breakout:long_board_socket -> zx_splicer:long_board_socket
- J3: footprint zx_bus_breakout:short_pin_header -> zx_splicer:short_pin_header
- J4: footprint zx_bus_breakout:long_pin_header -> zx_splicer:long_pin_header
- J5: footprint zx_bus_breakout:short_pin_socket -> zx_splicer:short_pin_socket
- J6: footprint zx_bus_breakout:long_pin_socket -> zx_splicer:long_pin_socket
- J7: footprint zx_bus_breakout:short_board_edge -> zx_splicer:short_board_edge
- J8: footprint zx_bus_breakout:long_board_edge -> zx_splicer:long_board_edge
Changed lines of the file:
@@
 EESchema Schematic File Version 4
-LIBS:zx_bus_breakout-cache
+LIBS:zx_splicer-cache
 EELAYER 30 0
 EELAYER END
@@
 F 0 "J1" H 3450 1917 50  0000 C CNN
 F 1 "Conn_02x04_Row_Letter_First" H 3450 1826 50  0000 C CNN
-F 2 "zx_bus_breakout:short_board_socket" H 3450 1825 50  0001 C CNN
+F 2 "zx_splicer:short_board_socket" H 3450 1825 50  0001 C CNN
 F 3 "~" H 3400 1600 50  0001 C CNN
 	1    3400 1600
@@
 F 0 "J2" H 3450 4567 50  0000 C CNN
 F 1 "Conn_02x23_Row_Letter_First" H 3450 4476 50  0000 C CNN
-F 2 "zx_bus_breakout:long_board_socket" H 3400 3250 50  0001 C CNN
+F 2 "zx_splicer:long_board_socket" H 3400 3250 50  0001 C CNN
 F 3 "" H 3400 3250 50  0001 C CNN
 	1    3400 3250
@@
 F 0 "J3" H 4950 1917 50  0000 C CNN
 F 1 "Conn_02x04_Row_Letter_First" H 4950 1826 50  0000 C CNN
-F 2 "zx_bus_breakout:short_pin_header" H 4900 1600 50  0001 C CNN
+F 2 "zx_splicer:short_pin_header" H 4900 1600 50  0001 C CNN
 F 3 "~" H 4900 1600 50  0001 C CNN
 	1    4900 1600
@@
 F 0 "J4" H 4950 4567 50  0000 C CNN
 F 1 "Conn_02x23_Row_Letter_First" H 4950 4476 50  0000 C CNN
-F 2 "zx_bus_breakout:long_pin_header" H 4900 3250 50  0001 C CNN
+F 2 "zx_splicer:long_pin_header" H 4900 3250 50  0001 C CNN
 F 3 "~" H 4900 3250 50  0001 C CNN
 	1    4900 3250
@@
 F 0 "J5" H 6450 1917 50  0000 C CNN
 F 1 "Conn_02x04_Row_Letter_First" H 6450 1826 50  0000 C CNN
-F 2 "zx_bus_breakout:short_pin_socket" H 6400 1600 50  0001 C CNN
+F 2 "zx_splicer:short_pin_socket" H 6400 1600 50  0001 C CNN
 F 3 "~" H 6400 1600 50  0001 C CNN
 	1    6400 1600
@@
 F 0 "J6" H 6450 4567 50  0000 C CNN
 F 1 "Conn_02x23_Row_Letter_First" H 6450 4476 50  0000 C CNN
-F 2 "zx_bus_breakout:long_pin_socket" H 6400 3250 50  0001 C CNN
+F 2 "zx_splicer:long_pin_socket" H 6400 3250 50  0001 C CNN
 F 3 "~" H 6400 3250 50  0001 C CNN
 	1    6400 3250
@@
 F 0 "J7" H 7950 1917 50  0000 C CNN
 F 1 "Conn_02x04_Row_Letter_First" H 7950 1826 50  0000 C CNN
-F 2 "zx_bus_breakout:short_board_edge" H 7900 1600 50  0001 C CNN
+F 2 "zx_splicer:short_board_edge" H 7900 1600 50  0001 C CNN
 F 3 "~" H 7900 1600 50  0001 C CNN
 	1    7900 1600
@@
 F 0 "J8" H 7950 4567 50  0000 C CNN
 F 1 "Conn_02x23_Row_Letter_First" H 7950 4476 50  0000 C CNN
-F 2 "zx_bus_breakout:long_board_edge" H 7900 3250 50  0001 C CNN
+F 2 "zx_splicer:long_board_edge" H 7900 3250 50  0001 C CNN
 F 3 "~" H 7900 3250 50  0001 C CNN
 	1    7900 3250
